Commit message: Remove mimic joint plugins and reproduce the mechanism with gazebo

File: xarm_gripper/urdf/xarm_gripper.gazebo.xacro (robot description, xacro)
@@ -51,5 +51,5 @@
     </gazebo>
     <gazebo reference="${prefix}left_outer_knuckle">
-      <selfCollide>false</selfCollide>
+      <selfCollide>true</selfCollide>
     </gazebo>
     <gazebo reference="${prefix}left_finger">
@@ -60,5 +60,5 @@
     </gazebo>
     <gazebo reference="${prefix}right_outer_knuckle">
-      <selfCollide>false</selfCollide>
+      <selfCollide>true</selfCollide>
     </gazebo>
     <gazebo reference="${prefix}right_finger">

File: xarm_gripper/urdf/xarm_gripper.urdf.xacro (robot description, xacro)
@@ -90,5 +90,33 @@
       </geometry>
     </collision>
-  </link>
+    <collision>
+      <geometry>
+        <mesh
+          scale="0.02 0.07 0.07"
+          filename="package://xarm_gripper/meshes/simple_gear_for_gripper.stl" />
+      </geometry>
+    </collision>
+  </link>
+  <gazebo>
+    <joint name="${prefix}left_loop_joint" type="revolute">
+      <parent>${prefix}left_inner_knuckle</parent>
+      <child>${prefix}left_finger</child>
+      <pose>0 -0.015 0.015 0 0 0</pose>
+      <axis>
+        <xyz>1 0 0</xyz>
+        <use_parent_model_frame>true</use_parent_model_frame>
+      </axis>
+      <physics>
+        <ode>
+          <implicit_spring_damper>1</implicit_spring_damper>
+          <cfm_damping>0</cfm_damping>
+          <limit>
+            <cfm>1e-7</cfm>
+            <erp>0.8</erp>
+          </limit>
+        </ode>
+      </physics>
+    </joint>
+  </gazebo>
   <joint
     name="${prefix}drive_joint"
@@ -265,5 +293,33 @@
       </geometry>
     </collision>
-  </link>
+    <collision>
+      <geometry>
+        <mesh
+          scale="0.02 0.07 0.07"
+          filename="package://xarm_gripper/meshes/simple_gear_for_gripper.stl" />
+      </geometry>
+    </collision>
+  </link>
+  <gazebo>
+    <joint name="${prefix}right_loop_joint" type="revolute">
+      <parent>${prefix}right_inner_knuckle</parent>
+      <child>${prefix}right_finger</child>
+      <pose>0 0.015 0.015 0 0 0</pose>
+      <axis>
+        <xyz>1 0 0</xyz>
+        <use_parent_model_frame>true</use_parent_model_frame>
+      </axis>
+      <physics>
+        <ode>
+          <implicit_spring_damper>1</implicit_spring_damper>
+          <cfm_damping>0</cfm_damping>
+          <limit>
+            <cfm>1e-7</cfm>
+            <erp>0.8</erp>
+          </limit>
+        </ode>
+      </physics>
+    </joint>
+  </gazebo>
   <joint
     name="${prefix}right_outer_knuckle_joint"

File: xarm_gripper/urdf/xarm_gripper_model.xacro (robot description, xacro)
@@ -15,20 +15,4 @@
     <xacro:xarm_gripper_gazebo prefix="${prefix}" />
     <xacro:xarm_gazebo_grasp_fix prefix="${prefix}" palm_link="${prefix}link${robot_dof}" />
-    <!-- mimic_joint_plugin has to be installed: -->
-    <xacro:mimic_joint_plugin_gazebo name_prefix="${prefix}left_finger_joint"
-      following_joint="${prefix}drive_joint" mimic_joint="${prefix}left_finger_joint"
-      has_pid="false" multiplier="1.0" max_effort="10.0" />
-    <xacro:mimic_joint_plugin_gazebo name_prefix="${prefix}left_inner_knuckle_joint"
-      following_joint="${prefix}drive_joint" mimic_joint="${prefix}left_inner_knuckle_joint"
-      has_pid="false" multiplier="1.0" max_effort="10.0" />
-    <xacro:mimic_joint_plugin_gazebo name_prefix="${prefix}right_outer_knuckle_joint"
-      following_joint="${prefix}drive_joint" mimic_joint="${prefix}right_outer_knuckle_joint"
-      has_pid="false" multiplier="1.0" max_effort="10.0" />
-    <xacro:mimic_joint_plugin_gazebo name_prefix="${prefix}right_finger_joint"
-      following_joint="${prefix}drive_joint" mimic_joint="${prefix}right_finger_joint"
-      has_pid="false" multiplier="1.0" max_effort="10.0" />
-    <xacro:mimic_joint_plugin_gazebo name_prefix="${prefix}right_inner_knuckle_joint"
-      following_joint="${prefix}drive_joint" mimic_joint="${prefix}right_inner_knuckle_joint"
-      has_pid="false" multiplier="1.0" max_effort="10.0" />
   </xacro:macro>
 </robot>

Commit message: Remove self-collision

File: xarm_gripper/urdf/xarm_gripper.gazebo.xacro (robot description, xacro)
@@ -51,5 +51,12 @@
     </gazebo>
     <gazebo reference="${prefix}left_outer_knuckle">
+      <kp>100000.0</kp>
+      <kd>100.0</kd>
+      <mu1>0</mu1>
+      <maxVel>1.0</maxVel>
+      <minDepth>0.0001</minDepth>
+      <maxContacts>16</maxContacts>
       <selfCollide>true</selfCollide>
+      <dampingFactor>0</dampingFactor>
     </gazebo>
     <gazebo reference="${prefix}left_finger">
@@ -60,5 +67,12 @@
     </gazebo>
     <gazebo reference="${prefix}right_outer_knuckle">
+      <kp>100000.0</kp>
+      <kd>100.0</kd>
+      <mu1>0</mu1>
+      <maxVel>1.0</maxVel>
+      <minDepth>0.0001</minDepth>
+      <maxContacts>16</maxContacts>
       <selfCollide>true</selfCollide>
+      <dampingFactor>0</dampingFactor>
     </gazebo>
     <gazebo reference="${prefix}right_finger">

File: xarm_gripper/urdf/xarm_gripper.urdf.xacro (robot description, xacro)
@@ -105,14 +105,8 @@
       <axis>
         <xyz>1 0 0</xyz>
-        <use_parent_model_frame>true</use_parent_model_frame>
       </axis>
       <physics>
         <ode>
           <implicit_spring_damper>1</implicit_spring_damper>
-          <cfm_damping>0</cfm_damping>
-          <limit>
-            <cfm>1e-7</cfm>
-            <erp>0.8</erp>
-          </limit>
         </ode>
       </physics>
@@ -229,12 +223,4 @@
       </material>
     </visual>
-    <collision>
-      <origin
-        xyz="0 0.016 0.02"
-        rpy="-0.7 0 0" />
-      <geometry>
-        <box size="0.027 0.012 0.061"/>
-      </geometry>
-    </collision>
   </link>
   <joint
@@ -308,14 +294,8 @@
       <axis>
         <xyz>1 0 0</xyz>
-        <use_parent_model_frame>true</use_parent_model_frame>
       </axis>
       <physics>
         <ode>
           <implicit_spring_damper>1</implicit_spring_damper>
-          <cfm_damping>0</cfm_damping>
-          <limit>
-            <cfm>1e-7</cfm>
-            <erp>0.8</erp>
-          </limit>
         </ode>
       </physics>
@@ -433,12 +413,4 @@
       </material>
     </visual>
-    <collision>
-      <origin
-        xyz="0 -0.016 0.02"
-        rpy="0.7 0 0" />
-      <geometry>
-        <box size="0.027 0.012 0.061"/>
-      </geometry>
-    </collision>
   </link>
   <joint
