Commit message: Upscale small inertials

File: xarm_gripper/urdf/xarm_gripper.urdf.xacro (robot description, xacro)
@@ -61,12 +61,12 @@
         rpy="0 0 0" />
       <mass
-        value="0.033618" />
-      <inertia
-        ixx="1.9111E-05"
-        ixy="-1.8803E-17"
-        ixz="-1.1002E-17"
-        iyy="6.6256E-06"
-        iyz="-7.3008E-06"
-        izz="1.3185E-05" />
+        value="0.1" />
+      <inertia
+        ixx="5.7284E-05"
+        ixy="0"
+        ixz="0"
+        iyy="1.9708E-05"
+        iyz="-2.1717E-05"
+        izz="3.9220E-05" />
     </inertial>
     <visual>
@@ -116,12 +116,12 @@
         rpy="0 0 0" />
       <mass
-        value="0.048304" />
-      <inertia
-        ixx="1.7493E-05"
-        ixy="-4.2156E-19"
-        ixz="6.9164E-18"
-        iyy="1.7225E-05"
-        iyz="4.6433E-06"
-        izz="5.1466E-06" />
+        value="0.1" />
+      <inertia
+        ixx="3.6214E-05"
+        ixy="0"
+        ixz="0"
+        iyy="3.5660E-05"
+        iyz="9.6127E-06"
+        izz="1.0655E-05" />
     </inertial>
     <visual>
@@ -180,12 +180,12 @@
         rpy="0 0 0" />
       <mass
-        value="0.0230125781256706" />
-      <inertia
-        ixx="6.09490024271906E-06"
-        ixy="6.06651326160071E-11"
-        ixz="7.19102670500635E-11"
-        iyy="6.01955084375188E-06"
-        iyz="-2.75316812991721E-06"
-        izz="5.07862004479903E-06" />
+        value="0.1" />
+      <inertia
+        ixx="2.6486E-05"
+        ixy="0"
+        ixz="0"
+        iyy="2.6158E-05"
+        iyz="-1.1864E-05"
+        izz="2.2069E-05" />
     </inertial>
     <visual>
@@ -236,12 +236,12 @@
         rpy="0 0 0" />
       <mass
-        value="0.033618" />
-      <inertia
-        ixx="1.9111E-05"
-        ixy="-1.8789E-17"
-        ixz="1.0986E-17"
-        iyy="6.6256E-06"
-        iyz="7.3008E-06"
-        izz="1.3185E-05" />
+        value="0.1" />
+      <inertia
+        ixx="5.7284E-05"
+        ixy="0"
+        ixz="0"
+        iyy="1.9708E-05"
+        iyz="2.1717E-05"
+        izz="3.9220E-05" />
     </inertial>
     <visual>
@@ -292,12 +292,12 @@
         rpy="0 0 0" />
       <mass
-        value="0.048304" />
-      <inertia
-        ixx="1.7493E-05"
-        ixy="-5.0014E-19"
-        ixz="-7.5079E-18"
-        iyy="1.7225E-05"
-        iyz="-4.6435E-06"
-        izz="5.1466E-06" />
+        value="0.1" />
+      <inertia
+        ixx="3.6214E-05"
+        ixy="0"
+        ixz="0"
+        iyy="3.5660E-05"
+        iyz="-9.6127E-06"
+        izz="1.0655E-05" />
     </inertial>
     <visual>
@@ -356,12 +356,12 @@
         rpy="0 0 0" />
       <mass
-        value="0.023013" />
-      <inertia
-        ixx="6.0949E-06"
-        ixy="-6.0665E-11"
-        ixz="7.191E-11"
-        iyy="6.0197E-06"
-        iyz="2.7531E-06"
-        izz="5.0784E-06" />
+        value="0.1" />
+      <inertia
+        ixx="2.6486E-05"
+        ixy="0"
+        ixz="0"
+        iyy="2.6158E-05"
+        iyz="1.1864E-05"
+        izz="2.2069E-05" />
     </inertial>
     <visual>
